File: kicad_project/dry_storage_cabinet_kicad.kicad_sch (KiCad schematic)
At the start: 0 parts

Commit message: 70% hardware, testing now
Parts:
- added BZ1: Buzzer, Buzzer_Beeper:Buzzer_12x9.5RM7.6, symbol Device:Buzzer
- added C1, C3: 100n, Capacitor_THT:C_Disc_D5.0mm_W2.5mm_P5.00mm, symbol Device:C
- added C2: 100u, Capacitor_THT:CP_Radial_D6.3mm_P2.50mm, symbol Device:C_Polarized
- added D1, D2: IN5822, Diode_THT:D_DO-201AD_P15.24mm_Horizontal, symbol Device:D
- added D3: RED, LED_THT:LED_D3.0mm, symbol Device:LED
- added D4: GREEN, LED_THT:LED_D3.0mm, symbol Device:LED
- added H1, H2, H3, H4: MountingHole, MountingHole:MountingHole_3.2mm_M3, symbol Mechanical:MountingHole
- added J1: Barrel_Jack_Switch, Connector_BarrelJack:BarrelJack_GCT_DCJ200-10-A_Horizontal, symbol Connector:Barrel_Jack_Switch
- added J2: LM2596, otter:LM2596-DC-DC, symbol Connector:Conn_01x04_Pin
- added J3, J4, J5: Screw_Terminal_01x02, TerminalBlock:TerminalBlock_MaiXu_MX126-5.0-02P_1x02_P5.00mm, symbol Connector:Screw_Terminal_01x02
- added J6: OLED_SSD1309, Connector_PinHeader_2.54mm:PinHeader_1x04_P2.54mm_Vertical, symbol Connector:Conn_01x04_Pin
- added J7: SHT30_1, TerminalBlock:TerminalBlock_MaiXu_MX126-5.0-04P_1x04_P5.00mm, symbol Connector:Screw_Terminal_01x04
- added J8: NTC_MF_52_103_10K, TerminalBlock:TerminalBlock_MaiXu_MX126-5.0-02P_1x02_P5.00mm, symbol Connector:Screw_Terminal_01x02
- added Q1, Q2, Q3: IRLZ44N, Package_TO_SOT_THT:TO-220-3_Vertical, symbol Transistor_FET:Q_NMOS_GDS
- added R2, R4, R6: 100k, Resistor_THT:R_Axial_DIN0207_L6.3mm_D2.5mm_P10.16mm_Horizontal, symbol Device:R
- added R7: 330, Resistor_THT:R_Axial_DIN0207_L6.3mm_D2.5mm_P10.16mm_Horizontal, symbol Device:R
- added R8: 100, Resistor_THT:R_Axial_DIN0207_L6.3mm_D2.5mm_P10.16mm_Horizontal, symbol Device:R
- added R9: 10k-1%, Resistor_THT:R_Axial_DIN0207_L6.3mm_D2.5mm_P10.16mm_Horizontal, symbol Device:R
- added SW1: EC11, Rotary_Encoder:RotaryEncoder_Alps_EC11E-Switch_Vertical_H20mm_MountingHoles, symbol Device:RotaryEncoder_Switch_MP
- added SW2: MTS_102, SW_MTS102:MTS102, symbol Switch:SW_SPDT
- added U2: STM32F411 BlackPill, WeAct_Black_Pill_V2.0:STM32F411_Black_Pill, symbol WeAct_Black_Pill_V2.0:STM32F411_Black_Pill
Connections:
- new net: D4.1 (K), R8.1
- new net: D3.1 (K), R7.1
- new net +12V: J1.1, SW2.2 (B)
- new net +12V_SW: D1.1 (K), D2.1 (K), J2.2 (Pin_2), J3.2 (Pin_2), J4.2 (Pin_2), J5.2 (Pin_2), SW2.1 (A)
- new net +3.3V: J6.2 (Pin_2), J7.4 (Pin_4), R9.2, U2.20 (3.3V)
- new net +5V: C1.1, C2.1, J2.3 (Pin_3), U2.40 (5V)
- new net ADC0_NTC: C3.1, J8.1 (Pin_1), R9.1, U2.26 (A0)
- new net BUZZER_PIN: BZ1.1 (+), U2.4 (B15)
- new net COLD_FAN-: D2.2 (A), J5.1 (Pin_1), Q3.2 (D)
- new net COLD_FAN_PWM: Q3.1 (G), R6.2, U2.33 (A7)
- new net ENCODER_BUTTON: SW1.S1, U2.12 (B4)
- new net ERROR_LED: D3.2 (A), U2.2 (B13)
- new net GND: BZ1.2 (-), C1.2, C2.2, C3.2, J1.2, J1.3, J2.1 (Pin_1), J2.4 (Pin_4), J6.1 (Pin_1), J7.3 (Pin_3), J8.2 (Pin_2), Q1.3 (S), Q2.3 (S), Q3.3 (S), R2.1, R4.1, R6.1, R7.2, R8.2, SW1.C, SW1.S2, U2.19 (G), U2.39 (G)
- new net HOT_FAN-: D1.2 (A), J4.1 (Pin_1), Q2.2 (D)
- new net HOT_FAN_ENABLE: Q2.1 (G), R4.2, U2.29 (A3)
- new net I2C1_SCL: J6.3 (Pin_3), J7.2 (Pin_2), U2.14 (B6)
- new net I2C1_SDA: J6.4 (Pin_4), J7.1 (Pin_1), U2.15 (B7)
- new net NORMAL_LED: D4.2 (A), U2.3 (B14)
- new net PELTIER-: J3.1 (Pin_1), Q1.2 (D)
- new net PELTIER_ENABLE: Q1.1 (G), R2.2, U2.28 (A2)
- new net TIMER2_ENCODER_A: SW1.A, U2.11 (B3)
- new net TIMER2_ENCODER_B: SW1.B, U2.10 (A15)
- no-connect marks 0 -> 26
Other:
- note added: "BUZZER"
- note added: "DISPLAY"
- note added: "DRIVER"
- note added: "ENCODER ROTARY"
- note added: "MCU"
- note added: "POWER"
- note added: "SENSOR"
